Commit message: camera integration

File: lbr_description/urdf/iiwa14/iiwa14.xacro (robot description, xacro)
@@ -8,5 +8,5 @@
     <!-- arguments -->
     <xacro:arg name="robot_name" default="lbr" />
-    <xacro:arg name="mode" default="true" />
+    <xacro:arg name="mode" default="mock" />
     <xacro:arg
         name="joint_limits_path"
@@ -38,3 +38,54 @@
         robot_name="$(arg robot_name)"
         joint_limits_path="$(arg joint_limits_path)" />
+    <!-- ENVIRONMENT CAMERA -->
+    <!-- Camera link definition -->
+    <link name="env_camera_link">
+        <visual>
+            <origin xyz="0 0 0" rpy="0 0 0"/>
+            <geometry>
+                <box size="0.05 0.05 0.05"/>
+            </geometry>
+            <material name="camera_material">
+                <color rgba="0.5 0.5 0.5 1.0"/>
+            </material>
+        </visual>
+        <collision>
+            <origin xyz="0 0 0" rpy="0 0 0"/>
+            <geometry>
+                <box size="0.05 0.05 0.05"/>
+            </geometry>
+        </collision>
+        <inertial>
+            <mass value="0.1"/>
+            <inertia ixx="0.0001" ixy="0" ixz="0" iyy="0.0001" iyz="0" izz="0.0001"/>
+        </inertial>
+    </link>
+    <!-- Fixed joint: camera at world position (0, 0, 2.5), pointing down -->
+    <joint name="env_camera_joint" type="fixed">
+        <parent link="world"/>
+        <child link="env_camera_link"/>
+        <origin xyz="0.0 0.0 3.5" rpy="0 1.5708 0"/>
+    </joint>
+    <!-- Gazebo sensor configuration for the camera -->
+    <gazebo reference="env_camera_link">
+        <sensor name="env_camera" type="camera">
+            <camera>
+                <horizontal_fov>1.047</horizontal_fov>
+                <image>
+                    <width>640</width>
+                    <height>480</height>
+                    <format>R8G8B8</format>
+                </image>
+                <clip>
+                    <near>0.1</near>
+                    <far>100</far>
+                </clip>
+            </camera>
+            <always_on>1</always_on>
+            <update_rate>30</update_rate>
+            <visualize>true</visualize>
+            <topic>env_camera/image_raw</topic>
+        </sensor>
+    </gazebo>
+    <!-- END ENVIRONMENT CAMERA -->
 </robot>
