Commit message: introducing hande

File: lbr_description/urdf/iiwa14/iiwa14.urdf.xacro (robot description, xacro)
@@ -296,4 +296,29 @@
         <link name="${robot_name}_link_ee">
         </link>
+        <ros2_control name="robotiq_ros2_control" type="system">
+            <hardware>
+                <plugin>gz_ros2_control/GazeboSimSystem</plugin>
+            </hardware>
+            <joint name="hande_left_finger_joint">
+                <command_interface name="position">
+                <param name="min">0.0</param>
+                <param name="max">0.025</param>
+                </command_interface>
+                <state_interface name="position">
+                <param name="initial_value">0.0</param>
+                </state_interface>
+                <state_interface name="velocity"/>
+            </joint>
+            <joint name="hande_right_finger_joint">
+                <command_interface name="position">
+                <param name="min">0.0</param>
+                <param name="max">0.025</param>
+                </command_interface>
+                <state_interface name="position">
+                <param name="initial_value">0.0</param>
+                </state_interface>
+                <state_interface name="velocity"/>
+            </joint>
+        </ros2_control>
     </xacro:macro>
 </robot>

File: lbr_description/urdf/iiwa14/iiwa14.xacro (robot description, xacro)
@@ -6,4 +6,5 @@
     <xacro:include filename="$(find lbr_description)/gazebo/lbr_gazebo.xacro" />
     <xacro:include filename="$(find lbr_description)/ros2_control/lbr_system_interface.xacro" />
+    <xacro:include filename="$(find robotiq_description)/urdf/robotiq_hand_e_macro.urdf.xacro" />
     <!-- arguments -->
     <xacro:arg name="robot_name" default="lbr" />
@@ -27,4 +28,7 @@
         <child link="$(arg robot_name)_link_0" />
     </joint>
+    <xacro:robotiq_hande prefix="" parent= "$(arg robot_name)_link_ee">
+        <origin xyz="0 0 0" rpy="0 0 0" />
+    </xacro:robotiq_hande>
     <!-- macros for gazebo / mock / hardware -->
     <xacro:lbr_gazebo robot_name="$(arg robot_name)" />

Commit message: added sim arg to fix the use gripper in real hardware

File: lbr_description/urdf/iiwa14/iiwa14.urdf.xacro (robot description, xacro)
@@ -10,4 +10,5 @@
         <xacro:property name="joint_damping" value="10.0" />
         <xacro:property name="joint_friction" value="0.1" />
+        <xacro:arg name="sim" default="false" />
         <!-- links and joints -->
         <link name="${robot_name}_link_0">
@@ -296,29 +297,31 @@
         <link name="${robot_name}_link_ee">
         </link>
-        <ros2_control name="robotiq_ros2_control" type="system">
-            <hardware>
-                <plugin>gz_ros2_control/GazeboSimSystem</plugin>
-            </hardware>
-            <joint name="hande_left_finger_joint">
-                <command_interface name="position">
-                <param name="min">-0.025</param>
-                <param name="max">0.025</param>
-                </command_interface>
-                <state_interface name="position">
-                <param name="initial_value">0.0</param>
-                </state_interface>
-                <state_interface name="velocity"/>
-            </joint>
-            <joint name="hande_right_finger_joint">
-                <command_interface name="position">
-                <param name="min">-0.025</param>
-                <param name="max">0.025</param>
-                </command_interface>
-                <state_interface name="position">
-                <param name="initial_value">0.0</param>
-                </state_interface>
-                <state_interface name="velocity"/>
-            </joint>
-        </ros2_control>
+        <xacro:if value="$(arg sim)">
+            <ros2_control name="robotiq_ros2_control" type="system">
+                <hardware>
+                    <plugin>gz_ros2_control/GazeboSimSystem</plugin>
+                </hardware>
+                <joint name="hande_left_finger_joint">
+                    <command_interface name="position">
+                    <param name="min">-0.025</param>
+                    <param name="max">0.025</param>
+                    </command_interface>
+                    <state_interface name="position">
+                    <param name="initial_value">0.0</param>
+                    </state_interface>
+                    <state_interface name="velocity"/>
+                </joint>
+                <joint name="hande_right_finger_joint">
+                    <command_interface name="position">
+                    <param name="min">-0.025</param>
+                    <param name="max">0.025</param>
+                    </command_interface>
+                    <state_interface name="position">
+                    <param name="initial_value">0.0</param>
+                    </state_interface>
+                    <state_interface name="velocity"/>
+                </joint>
+            </ros2_control>
+        </xacro:if>
     </xacro:macro>
 </robot>
